File: hardware/kicad/rak4630_interface.kicad_sch (KiCad schematic)
At the start: 21 parts, among them IC1 RAK4630, J1 UJ20-C-H-G-SMT-5-P16-TR, J2 Conn_01x08_Pin, J3 Conn_01x08_Pin, SW1 RESET, U1 TLV62569DBV, U2 TPD2EUSB30

Commit message: update pcb
Connections:
- net UART1_RX: now also IC1.9 (P0.19/UART1_RX_(AT_COMMAND)); no longer IC1.8 (P0.17/UART2_DE)
- net UART1_TX: now also IC1.10 (P0.20/UART1_TX_(AT_COMMAND)); no longer IC1.9 (P0.19/UART1_RX_(AT_COMMAND))
Changed lines of the file:
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@@
 	(wire
 		(pts
-			(xy 78.74 72.39) (xy 88.9 72.39)
+			(xy 78.74 74.93) (xy 88.9 74.93)
 		)
 		(stroke
@@
 	(wire
 		(pts
-			(xy 78.74 74.93) (xy 88.9 74.93)
+			(xy 78.74 78.74) (xy 88.9 78.74)
 		)
 		(stroke
@@
 	)
 	(label "UART1_TX"
-		(at 78.74 74.93 0)
+		(at 78.74 78.74 0)
 		(effects
 			(font
@@
 	)
 	(label "UART1_RX"
-		(at 78.74 72.39 0)
+		(at 78.74 74.93 0)
 		(effects
 			(font

Commit message: update pcb
Parts:
- added J4: Conn_01x03_Pin, Connector_PinSocket_2.54mm:PinSocket_1x03_P2.54mm_Vertical, symbol Connector:Conn_01x03_Pin
Connections:
- net GND: now also SW1.2, J4.3 (Pin_3); no longer SW1.1
- net RESET: now also SW1.1; no longer SW1.2
- net SWD_CLK: now reaches IC1.18 (SWDCLK)
- net SWD_CLK: now also J4.1 (Pin_1)
- net SWD_IO: now reaches IC1.19 (SWDIO)
- net SWD_IO: now also J4.2 (Pin_2)
Other:
- moved on the sheet: J2, J3, JP1

Commit message: update annotations
Other:
- company: (none) -> pashamray
- title: (none) -> RAK4630 Interface
Changed lines of the file:
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@@
 	(generator_version "9.0")
 	(paper "A4")
+	(title_block
+		(title "RAK4630 Interface")
+		(date "2026-04-10")
+		(rev "1.0.0")
+		(company "pashamray")
+	)
 	(text "Vout = Vfb (1 + R_VOUT / R_FB)\n3.3 = 0.6 (1 + 450000 / 100000)"
 		(exclude_from_sim no)
