File: hardware/kicad/rak4630_interface.kicad_pcb (KiCad board)
At the start: 2 copper layers, 50.8 x 30.5 mm, 25 parts, among them IC1 RAK4630, J1 UJ20-C-H-G-SMT-5-P16-TR, J2 Conn_01x08_Pin, J3 Conn_01x08_Pin, SW1 RESET, U1 TLV62569DBV, U2 TPD2EUSB30

Commit message: update pcb
Connections:
- IC1 pad 10: unconnected-(IC1-P0.20/UART1_TX_(AT_COMMAND)-Pad10) -> /UART1_TX
- IC1 pad 8: /UART1_RX -> unconnected-(IC1-P0.17/UART2_DE-Pad8)
- IC1 pad 9: /UART1_TX -> /UART1_RX
Routing:
- net /UART1_RX: track 7.37 -> 7.95 mm

Commit message: update pcb
Parts:
- added J4: Conn_01x03_Pin, Connector_PinSocket_2.54mm:PinSocket_1x03_P2.54mm_Vertical, F.Cu at (170.5, 79.4)
- added REF**: OSHW-Logo2_7.3x6mm_SilkScreen, Symbol:OSHW-Logo2_7.3x6mm_SilkScreen, B.Cu at (155.1, 81.7)
- moved TP3 37.1 mm to (137.3, 92.5)
- moved SW1 7.86 mm to (170.4, 88.5)
- moved C5 0.52 mm to (170.3, 83.5)
Connections:
- IC1 pad 18: unconnected-(IC1-SWDCLK-Pad18) -> /SWD_CLK
- IC1 pad 19: unconnected-(IC1-SWDIO-Pad19) -> /SWD_IO
- SW1 pad 1: GND -> /RESET
- SW1 pad 2: /RESET -> GND
Routing:
- net /SWD_IO: track 0.00 -> 5.28 mm
- net /SWD_CLK: track 0.00 -> 4.72 mm
- net VBAT: track 37.5 -> 42.1 mm, vias 0 -> 2
- net /RESET: track 5.69 -> 8.65 mm
Other:
- board text added: "https://github.com/pashamray/rak4630_interface"

Commit message: update pcb
Routing:
- net VDD: track 58.4 -> 56.2 mm
- net VBAT: track 42.1 -> 41.4 mm
Other:
- board text added: "GND"
- board text added: "I2C SCL"
- board text added: "I2C SDA"
- board text added: "LED1"
- board text added: "LED2"
- board text added: "Rev.: 1.0.0"
- board text added: "SW1"
- board text added: "SW2"
- board text added: "SWD CLK"
- board text added: "SWD IO"
- board text added: "UART1 RX"
- board text added: "UART1 TX"
- board text added: "UART2 RX"
- board text added: "UART2 TX"
- board text added: "VDD"
