File: hardware/kicad/rak4630_interface.kicad_pcb (KiCad board)
At the start: 2 copper layers, 50.8 x 30.5 mm, 27 parts, among them IC1 RAK4630, J1 UJ20-C-H-G-SMT-5-P16-TR, J2 Conn_01x08_Pin, J3 Conn_01x08_Pin, J4 Conn_01x03_Pin, SW1 RESET, U1 TLV62569DBV, U2 TPD2EUSB30

Commit message: update pcb
Other:
- board text added: "RAK4630 Interface Rev.: 1.0.0"
- board text removed: "Rev.: 1.0.0"
Changed lines of the file:
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@@
 		)
 	)
-	(gr_text "Rev.: 1.0.0"
-		(at 134.005 94.1 0)
+	(gr_text "RAK4630 Interface\nRev.: 1.0.0"
+		(at 138.069 69.843 0)
 		(layer "B.SilkS" knockout)
 		(effects
